File: output/Output_stage.kicad_pcb (KiCad board)
At the start: 2 copper layers, 64.8 x 27.9 mm, 8 parts, among them J1 Conn_01x03_Socket, J2 Conn_01x02_Socket, J3 Conn_01x02_Socket, Q1 BTA41-600B, U1 MOC3041M

Commit message: Some tuning
Parts:
- added REF**: TestPoint_THTPad_D3.0mm_Drill1.5mm, TestPoint:TestPoint_THTPad_D3.0mm_Drill1.5mm, F.Cu at (54.4, 42.7)
- added REF**: TestPoint_THTPad_D3.0mm_Drill1.5mm, TestPoint:TestPoint_THTPad_D3.0mm_Drill1.5mm, F.Cu at (53.8, 35.8)
- added REF**: TestPoint_THTPad_D3.0mm_Drill1.5mm, TestPoint:TestPoint_THTPad_D3.0mm_Drill1.5mm, F.Cu at (43.2, 42.7)
- added REF**: TestPoint_THTPad_D3.0mm_Drill1.5mm, TestPoint:TestPoint_THTPad_D3.0mm_Drill1.5mm, F.Cu at (45.7, 35.8)
- J2, J3: value Conn_01x02_Socket -> Control/LED
- Q1: value BTA41-600B -> BTA41
- moved Q1 1.27 mm to (47.9, 31.8)
- moved R2 1.27 mm to (63.5, 50.8)
- moved J3 0.11 mm to (94.6, 49.0)
Connections:
- net Net-(J1-Pin_1) renamed LINE
- net Net-(J1-Pin_3) renamed S/LINE
Routing:
- net Net-(Q1-G): track 24.3 -> 26.1 mm
- net LINE: track 33.0 -> 34.3 mm
- net S/LINE: track 44.6 -> 45.4 mm
- added copper zone on B.Cu, net LINE
- added copper zone on B.Cu, net S/LINE
Other:
- outline, holes or cut-outs redrawn

Commit message: Tuning + labels
Parts:
- added kibuzzard-6431D11C: G***, kibuzzard-6431D11C, F.Cu at (39.6, 41.9)
- added kibuzzard-6431D738: G***, kibuzzard-6431D738, F.Cu at (78.0, 48.0)
- moved R2 3.58 mm to (65.2, 47.6)
- moved REF** 3.18 mm to (46.4, 42.5)
- moved REF** 2.79 mm to (48.5, 35.8)
- moved J1 2.54 mm to (55.9, 48.9)
- moved R3 2.25 mm to (69.8, 33.4)
- moved U1 2.08 mm to (83.2, 39.6)
- moved REF** 2.03 mm to (55.9, 35.8)
- moved Q1 1.91 mm to (49.8, 31.8)
- moved REF** 1.53 mm to (55.9, 42.5)
- moved J2 0.76 mm to (95.4, 40.0)
- moved J3 0.76 mm to (95.4, 49.0)
Routing:
- net LINE: track 34.3 -> 17.3 mm
- net S/LINE: track 45.4 -> 29.2 mm
- net Net-(J2-Pin_2): track 22.4 -> 18.0 mm
- net Net-(R1-Pad2): track 11.6 -> 8.51 mm
- net Net-(Q1-G): track 26.1 -> 24.8 mm
- net Net-(J2-Pin_1): track 19.3 -> 18.8 mm
Other:
- outline, holes or cut-outs redrawn
- board text added: "+"
