File: 3-phase/mainboard/3phaseDiverter-rounded.kicad_pcb (KiCad board)
At the start: 2 copper layers, 144.8 x 120.6 mm, 99 parts, among them CN9 SMA, IC1 ATmega328-P, IC2 LM358, J0 FTDI, J1 RESET, J10 D10, J11 D11, J12 D12, J13 D13, J14 +5V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

Commit message: Tuning
Routing:
- net UnregDC+: track 193.6 -> 192.9 mm
- net GND: vias 84 -> 180
- net Earth: vias 0 -> 9

Commit message: PCB tuning
Parts:
- added G***: LOGO, LOGO, F.Cu at (54.0, 71.5)
Routing:
- net GND: vias 180 -> 185

Commit message: Some tuning
Parts:
- IC1: footprint Package_DIP:DIP-28_W7.62mm_Socket_LongPads -> PCM_Package_DIP_AKL:DIP-28_W7.62mm_Socket_LongPads
- IC2: footprint Package_DIP:DIP-8_W7.62mm_Socket_LongPads -> PCM_Package_DIP_AKL:DIP-8_W7.62mm_Socket_LongPads
- moved C6 0.26 mm to (90.3, 38.8)
Routing:
- net /D2: track 34.7 -> 35.3 mm
- net GND: vias 185 -> 184

Commit message: Some updates
Parts:
- added REF**: Symbol_HighVoltage_Type2_Silk_VerySmall, Library:Symbol_HighVoltage_Type2_Silk_VerySmall, F.Cu at (108.7, 121.4)
- added REF**: Symbol_HighVoltage_Type2_Silk_VerySmall, Library:Symbol_HighVoltage_Type2_Silk_VerySmall, F.Cu at (63.3, 121.4)
- added REF**: Symbol_HighVoltage_Type2_Silk_VerySmall, Library:Symbol_HighVoltage_Type2_Silk_VerySmall, B.Cu at (135.2, 124.5)
- added REF**: Symbol_HighVoltage_Type2_Silk_VerySmall, Library:Symbol_HighVoltage_Type2_Silk_VerySmall, B.Cu at (87.0, 124.5)
- added REF**: Symbol_HighVoltage_Type2_Silk_VerySmall, Library:Symbol_HighVoltage_Type2_Silk_VerySmall, B.Cu at (38.6, 124.5)
- added kibuzzard-6431D11C: G***, kibuzzard-6431D11C, F.Cu at (69.2, 74.1)
- added kibuzzard-64EB6544: G***, kibuzzard-64EB6544, F.Cu at (68.5, 78.4)
- moved G*** 7.84 mm to (46.6, 69.1)
Routing:
- net GND: vias 184 -> 185
