File: 3-phase/mainboard/3phaseDiverter.kicad_pcb (KiCad board)
At the start: 2 copper layers, 144.8 x 120.6 mm, 110 parts, among them CN9 SMA, IC1 ATmega328-P, IC2 LM358, J0 FTDI, J1 RESET, J10 D10, J11 D11, J12 D12, J13 D13, J14 +5V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

Commit message: Tuning
Routing:
- net +3.3V: track 204.9 -> 202.7 mm
- net Net-(R14-Pad2): track 29.0 -> 27.3 mm
- net Net-(IC1-AREF): track 5.08 -> 3.77 mm
- net /D2: track 36.4 -> 35.6 mm
- net /D10: track 48.5 -> 47.7 mm
- net Net-(CN9-Pad1): track 8.21 -> 7.48 mm
- net TX: track 35.1 -> 34.4 mm
- net /D5: track 37.5 -> 36.9 mm
- net RX: track 32.3 -> 31.7 mm
- net /D12: track 90.6 -> 91.1 mm
- net /D6: track 32.5 -> 32.0 mm
- net AVCC: track 173.9 -> 173.3 mm

Commit message: Upd PCB V4.0
Parts:
- removed kibuzzard-65314627: G***, kibuzzard-65314627
- added J16: D2, Library:Molex_SL_171971-0002_1x02_P2.54mm_Vertical, F.Cu at (112.1, 31.8)
- added J17: D3, Library:Molex_SL_171971-0002_1x02_P2.54mm_Vertical, F.Cu at (104.4, 31.8)
- added J18: D4, Library:Molex_SL_171971-0002_1x02_P2.54mm_Vertical, F.Cu at (96.8, 31.8)
- added J19: D5, Library:Molex_SL_171971-0002_1x02_P2.54mm_Vertical, F.Cu at (89.2, 31.8)
- added J21: D6, Library:Molex_SL_171971-0002_1x02_P2.54mm_Vertical, F.Cu at (81.6, 31.8)
- added J22: D7, Library:Molex_SL_171971-0002_1x02_P2.54mm_Vertical, F.Cu at (74.0, 31.8)
- added J23: D8, Library:Molex_SL_171971-0002_1x02_P2.54mm_Vertical, F.Cu at (66.3, 31.8)
- added J24: D9, Library:Molex_SL_171971-0002_1x02_P2.54mm_Vertical, F.Cu at (58.7, 31.8)
- added J25: D10, Library:Molex_SL_171971-0002_1x02_P2.54mm_Vertical, F.Cu at (51.1, 31.8)
- added J26: D11, Library:Molex_SL_171971-0002_1x02_P2.54mm_Vertical, F.Cu at (43.5, 31.8)
- added J27: D12, Library:Molex_SL_171971-0002_1x02_P2.54mm_Vertical, F.Cu at (35.9, 31.8)
- added J28: D13, Library:Molex_SL_171971-0002_1x02_P2.54mm_Vertical, F.Cu at (28.3, 31.8)
- added kibuzzard-653D8BA7: G***, kibuzzard-653D8BA7, F.Cu at (17.3, 77.2)
- TP1: value Test Vref -> Vref
- TP2: value Test VCC -> VCC
- TP3: value Test GND -> GND
- moved C3 115.1 mm to (20.8, 56.7)
- moved C5 115.0 mm to (20.8, 61.8), turned to -90 degrees
- moved VR2 114.0 mm to (23.3, 51.4), turned to 180 degrees
- moved G*** 58.1 mm to (104.4, 73.7)
- moved TP3 22.0 mm to (107.5, 43.8)
- moved kibuzzard-6431D11C 16.2 mm to (52.5, 68.9)
- moved kibuzzard-64EB6544 16.2 mm to (52.9, 73.5)
- moved kibuzzard-64EB6544 16.0 mm to (53.5, 72.2)
- moved kibuzzard-6431D11C 15.9 mm to (54.2, 68.2)
- moved C6 7.43 mm to (134.4, 36.4)
- moved J1 7.43 mm to (123.8, 42.6)
- moved R1 7.43 mm to (132.9, 21.5)
- moved J0 7.43 mm to (123.7, 34.1)
- moved R22 7.43 mm to (129.8, 21.5)
- moved TP2 6.12 mm to (130.0, 50.5)
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Routing:
- net +3.3V: track 202.7 -> 36.0 mm
- net VCC: track 276.3 -> 305.7 mm
- net /D12: track 91.1 -> 70.7 mm
- net /D2: track 35.6 -> 47.6 mm
- net Net-(JP3-B): track 65.4 -> 53.5 mm
- net /D5: track 36.9 -> 46.8 mm
- net TX: track 34.4 -> 43.7 mm
- net /D3: track 27.7 -> 36.3 mm
- net RX: track 31.7 -> 39.7 mm
- net /D6: track 32.0 -> 39.4 mm
- net VREF: track 201.4 -> 194.0 mm
- net RESET: track 40.1 -> 47.3 mm
- net /D10: track 47.7 -> 54.7 mm
- net /D11: track 59.5 -> 65.8 mm
- net AVCC: track 173.3 -> 167.3 mm
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Other:
- board text added: "<GND"
- board text added: "ANT"
- board text added: "CLK"
- board text added: "FFS"
- board text added: "FFTI"
- board text added: "GND"
- board text added: "GND>"
- board text added: "IRQ"
- board text added: "RST"
- board text added: "SCK"
- board text added: "SD0"
- board text added: "SDI"
- board text added: "SEL"
- board text added: "VDD"
- board text added: "nINT"

Commit message: Update
Parts:
- moved J1 19.3 mm to (123.7, 23.3)
- moved J0 7.82 mm to (123.7, 41.9)
Routing:
- net Net-(J0-DTR): track 26.1 -> 19.4 mm
- net TX: track 43.7 -> 38.1 mm
- net RX: track 39.7 -> 34.7 mm
- net Net-(IC1-AREF): track 4.51 -> 3.74 mm
- net /D2: track 47.6 -> 47.0 mm
Changed lines of the file:
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@@
   )
   (footprint "Library:Molex_SL_171971-0006_1x06_P2.54mm_Vertical" (layer "F.Cu")
-    (at 123.749996 34.1122 90)
+    (at 123.719996 41.93 90)
     (descr "Molex Stackable Linear Connector, 171971-0006 (compatible alternatives: 171971-0106, 171971-0206), 6 Pins per row (https://www.molex.com/pdm_docs/sd/1719710002_sd.pdf), generated with kicad-footprint-generator")
     (tags "connector Molex SL vertical")
@@
         (effects (font (size 1 1) (thickness 0.15)))
     )
-    (fp_text value "FTDI" (at 16.3322 0 180) (layer "F.SilkS")
+    (fp_text value "FTDI" (at 6.35 -3.649996 90) (layer "F.SilkS")
         (effects (font (size 1 1) (thickness 0.15)))
     )
@@
     (attr board_only exclude_from_pos_files exclude_from_bom)
     (fp_text reference "kibuzzard-653D8BA7" (at 0 -4.549378 -90) (layer "F.SilkS") hide
-        (effects (font (size 0 0)))
+        (effects (font (size 0 0) (thickness 0.15)))
     )
     (fp_text value "G***" (at 0 4.549378 -90) (layer "F.SilkS") hide
-        (effects (font (size 0 0)))
+        (effects (font (size 0 0) (thickness 0.15)))
     )
     (fp_poly
@@
   )
   (footprint "Library:Molex_SL_171971-0002_1x02_P2.54mm_Vertical" (layer "F.Cu")
-    (at 123.7634 42.6212 90)
+    (at 123.72 23.3 90)
     (descr "Molex Stackable Linear Connector, 171971-0002 (compatible alternatives: 171971-0102, 171971-0202), 2 Pins per row (https://www.molex.com/pdm_docs/sd/1719710002_sd.pdf), generated with kicad-footprint-generator")
     (tags "connector Molex SL vertical")
@@
         (effects (font (size 1 1) (thickness 0.15)))
     )
-    (fp_text value "RESET" (at 1.27 5.25 90) (layer "F.SilkS")
+    (fp_text value "RESET" (at 6 -0.02 180) (layer "F.SilkS")
         (effects (font (size 1 1) (thickness 0.15)))
     )
@@
     (effects (font (size 1 1) (thickness 0.15)) (justify right))
   )
-  (gr_text "GND>" (at 118.9228 34.1122) (layer "F.SilkS")
+  (gr_text "GND>" (at 118.9228 41.93) (layer "F.SilkS")
     (effects (font (size 1 1) (thickness 0.15)))
   )
@@
   (segment (start 136.437401 95.6818) (end 139.942601 99.187) (width 1) (layer "F.Cu") (net 9))
   (segment (start 139.942601 99.187) (end 151.5186 99.187) (width 1) (layer "F.Cu") (net 9))
-  (segment (start 82.0166 58.663195) (end 82.0166 58.8918) (width 0.5) (layer "F.Cu") (net 10))
   (segment (start 79.375 56.021595) (end 82.0166 58.663195) (width 0.5) (layer "F.Cu") (net 10))
-  (segment (start 79.375 55.4736) (end 79.375 56.021595) (width 0.5) (layer "F.Cu") (net 10))
-  (segment (start 129.366 36.3728) (end 127.3956 36.3728) (width 0.5) (layer "F.Cu") (net 11))
-  (segment (start 130.3166 35.4222) (end 130.3166 34.1376) (width 0.5) (layer "F.Cu") (net 11))
-  (segment (start 125.2112 21.3614) (end 123.749996 21.3614) (width 0.5) (layer "F.Cu") (net 11))
-  (segment (start 127.6496 23.7998) (end 125.2112 21.3614) (width 0.5) (layer "F.Cu") (net 11))
-  (segment (start 127.6496 29.464) (end 127.6496 23.7998) (width 0.5) (layer "F.Cu") (net 11))
-  (segment (start 127.3956 36.3728) (end 123.7634 40.005) (width 0.5) (layer "F.Cu") (net 11))
-  (segment (start 129.834 31.6484) (end 127.6496 29.464) (width 0.5) (layer "F.Cu") (net 11))
-  (segment (start 129.366 36.3728) (end 130.3166 35.4222) (width 0.5) (layer "F.Cu") (net 11))
-  (segment (start 129.834 33.655) (end 129.834 31.6484) (width 0.5) (layer "F.Cu") (net 11))
-  (segment (start 130.3166 34.1376) (end 129.834 33.655) (width 0.5) (layer "F.Cu") (net 11))
-  (segment (start 23.4442 73.1266) (end 23.46452 73.10628) (width 0.5) (layer "F.Cu") (net 12))
+  (segment (start 129.834 31.6484) (end 129.834 35.9048) (width 0.5) (layer "F.Cu") (net 11))
+  (segment (start 129.834 35.9048) (end 129.366 36.3728) (width 0.5) (layer "F.Cu") (net 11))
+  (segment (start 123.72 20.76) (end 125.55 20.76) (width 0.5) (layer "F.Cu") (net 11))
+  (segment (start 127.6496 22.8596) (end 127.6496 29.464) (width 0.5) (layer "F.Cu") (net 11))
+  (segment (start 127.6496 29.464) (end 129.834 31.6484) (width 0.5) (layer "F.Cu") (net 11))
+  (segment (start 125.55 20.76) (end 127.6496 22.8596) (width 0.5) (layer "F.Cu") (net 11))
   (segment (start 23.46452 73.10628) (end 23.46452 68.90512) (width 0.5) (layer "F.Cu") (net 12))
   (segment (start 23.46452 68.90512) (end 27.26944 65.1002) (width 0.5) (layer "F.Cu") (net 12))
@@
   (segment (start 40.3098 81.4916) (end 37.9392 79.121) (width 1) (layer "B.Cu") (net 13))
   (segment (start 69.8246 83.1596) (end 65.786 79.121) (width 1) (layer "B.Cu") (net 13))
-  (segment (start 40.3098 81.448096) (end 40.3098 81.4916) (width 1) (layer "B.Cu") (net 13))
   (segment (start 42.636896 79.121) (end 40.3098 81.448096) (width 1) (layer "B.Cu") (net 13))
   (segment (start 73.8632 79.121) (end 85.234 79.121) (width 1) (layer "B.Cu") (net 13))
@@
   (segment (start 116.84 83.185) (end 120.904 79.121) (width 1) (layer "B.Cu") (net 13))
   (segment (start 85.234 79.121) (end 87.6046 81.4916) (width 1) (layer "B.Cu") (net 13))
-  (segment (start 87.6046 81.448096) (end 87.6046 81.4916) (width 1) (layer "B.Cu") (net 13))
   (segment (start 113.03 79.121) (end 113.03 79.375) (width 1) (layer "B.Cu") (net 13))
   (segment (start 89.906296 79.1464) (end 87.6046 81.448096) (width 1) (layer "B.Cu") (net 13))
@@
   (segment (start 121.4374 122.4026) (end 121.4374 115.681801) (width 0.5) (layer "B.Cu") (net 21))
   (segment (start 41.78 130.0875) (end 48.26 130.0875) (width 0.5) (layer "B.Cu") (net 22))
-  (segment (start 119.875898 28.612502) (end 121.9962 26.4922) (width 0.5) (layer "F.Cu") (net 23))
-  (segment (start 94.615 47.8536) (end 94.615 47.757204) (width 0.5) (layer "F.Cu") (net 23))
-  (segment (start 102.570404 39.8018) (end 111.4806 39.8018) (width 0.5) (layer "F.Cu") (net 23))
-  (segment (start 119.875898 31.406502) (end 119.875898 28.612502) (width 0.5) (layer "F.Cu") (net 23))
-  (segment (start 121.9962 26.4922) (end 123.749996 26.4922) (width 0.5) (layer "F.Cu") (net 23))
-  (segment (start 94.615 47.757204) (end 102.570404 39.8018) (width 0.5) (layer "F.Cu") (net 23))
-  (segment (start 111.4806 39.8018) (end 119.875898 31.406502) (width 0.5) (layer "F.Cu") (net 23))
-  (segment (start 116.84 27.8638) (end 120.7516 23.9522) (width 0.5) (layer "F.Cu") (net 24))
-  (segment (start 92.075 47.2948) (end 101.9556 37.4142) (width 0.5) (layer "F.Cu") (net 24))
-  (segment (start 101.9556 37.4142) (end 110.287996 37.4142) (width 0.5) (layer "F.Cu") (net 24))
-  (segment (start 92.075 47.8536) (end 92.075 47.2948) (width 0.5) (layer "F.Cu") (net 24))
-  (segment (start 120.7516 23.9522) (end 123.749996 23.9522) (width 0.5) (layer "F.Cu") (net 24))
-  (segment (start 110.287996 37.4142) (end 116.84 30.862196) (width 0.5) (layer "F.Cu") (net 24))
-  (segment (start 116.84 30.862196) (end 116.84 27.8638) (width 0.5) (layer "F.Cu") (net 24))
+  (segment (start 116.9724 34.31) (end 111.4806 39.8018) (width 0.5) (layer "F.Cu") (net 23))
+  (segment (start 123.719996 34.31) (end 116.9724 34.31) (width 0.5) (layer "F.Cu") (net 23))
+  (segment (start 102.570404 39.8018) (end 94.615 47.757204) (width 0.5) (layer "F.Cu") (net 23))
+  (segment (start 111.4806 39.8018) (end 102.570404 39.8018) (width 0.5) (layer "F.Cu") (net 23))
+  (segment (start 110.287996 37.4142) (end 101.9556 37.4142) (width 0.5) (layer "F.Cu") (net 24))
+  (segment (start 115.932196 31.77) (end 110.287996 37.4142) (width 0.5) (layer "F.Cu") (net 24))
+  (segment (start 101.9556 37.4142) (end 92.075 47.2948) (width 0.5) (layer "F.Cu") (net 24))
+  (segment (start 123.719996 31.77) (end 115.932196 31.77) (width 0.5) (layer "F.Cu") (net 24))
   (segment (start 109.9058 29.2862) (end 112.060566 29.2862) (width 0.5) (layer "F.Cu") (net 25))
-  (segment (start 89.535 47.8536) (end 89.535 47.1932) (width 0.5) (layer "F.Cu") (net 25))
   (segment (start 108.7374 33.1216) (end 108.7374 30.4546) (width 0.5) (layer "F.Cu") (net 25))
   (segment (start 112.060566 20.8026) (end 113.380566 22.1226) (width 0.5) (layer "F.Cu") (net 25))
@@
   (segment (start 54.5338 64.2366) (end 61.5442 64.2366) (width 0.5) (layer "F.Cu") (net 36))
   (segment (start 24.4602 47.0154) (end 34.3408 56.896) (width 0.5) (layer "F.Cu") (net 36))
-  (segment (start 74.295 55.6006) (end 74.295 55.4736) (width 0.5) (layer "F.Cu") (net 36))
   (segment (start 28.250453 29.2862) (end 30.5308 29.2862) (width 0.5) (layer "F.Cu") (net 36))
   (segment (start 65.659 64.2366) (end 74.295 55.6006) (width 0.5) (layer "F.Cu") (net 36))
@@
   (segment (start 24.4348 62.9412) (end 24.4348 60.8076) (width 0.5) (layer "F.Cu") (net 61))
   (segment (start 20.7772 61.7982) (end 20.7772 63.5508) (width 0.5) (layer "F.Cu") (net 61))
-  (segment (start 29.27096 65.1002) (end 29.24556 65.1256) (width 0.5) (layer "F.Cu") (net 61))
   (segment (start 20.7772 51.3588) (end 20.7772 56.6928) (width 0.5) (layer "F.Cu") (net 61))
   (segment (start 29.24556 65.1256) (end 29.24556 69.55536) (width 0.5) (layer "F.Cu") (net 61))
@@
   (segment (start 78.9686 58.8918) (end 76.835 56.7582) (width 1) (layer "F.Cu") (net 62))
   (segment (start 60.6552 76.962) (end 60.6552 88.2142) (width 1) (layer "F.Cu") (net 62))
-  (segment (start 78.740005 58.699395) (end 78.740005 58.6886) (width 1) (layer "F.Cu") (net 62))
-  (segment (start 108.0516 76.6318) (end 108.072389 76.652589) (width 1) (layer "F.Cu") (net 62))
   (segment (start 108.072389 87.202811) (end 107.0356 88.2396) (width 1) (layer "F.Cu") (net 62))
   (segment (start 108.072389 76.652589) (end 108.072389 87.202811) (width 1) (layer "F.Cu") (net 62))
-  (segment (start 73.4314 65.470395) (end 73.431405 65.4704) (width 1) (layer "F.Cu") (net 62))
   (segment (start 76.835 56.7582) (end 76.835 55.4736) (width 1) (layer "F.Cu") (net 62))
   (via (at 108.0516 76.7334) (size 1.2) (drill 0.8) (layers "F.Cu" "B.Cu") (net 62))

Commit message: Update
Parts:
- removed kibuzzard-653D8BA7: G***, kibuzzard-653D8BA7
- added kibuzzard-653ECDA3: G***, kibuzzard-653ECDA3, F.Cu at (17.3, 77.2)
- moved R11 2.87 mm to (104.3, 62.9)
- moved C21 0.95 mm to (146.9, 68.2)
- moved C4 0.80 mm to (140.4, 38.0)
- moved J30 0.61 mm to (143.0, 45.9)
- moved C20 0.17 mm to (146.9, 64.7)
Routing:
- net Net-(J0-DTR): track 19.4 -> 26.5 mm
- net /D8: track 29.1 -> 35.5 mm
- net /D9: track 38.7 -> 44.0 mm
- net /D7: track 32.3 -> 37.2 mm
- net /D6: track 39.4 -> 42.8 mm
- net /D5: track 46.8 -> 49.8 mm
- net +5V: track 48.1 -> 45.5 mm
- net Net-(IC2A-+): track 25.2 -> 22.6 mm
- net /D10: track 54.7 -> 57.3 mm
- net /D11: track 65.8 -> 67.6 mm
- net /D2: track 47.0 -> 48.7 mm
- net /D4: track 34.0 -> 35.7 mm
- net /D3: track 36.3 -> 38.0 mm
- net /D12: track 70.7 -> 72.5 mm
- net /D13: track 93.8 -> 95.6 mm
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
Commit message: Update
Parts:
- TP4: value Test +3.3V -> +3.3V
- moved TP3 1.08 mm to (106.4, 43.8)
- moved TP4 0.83 mm to (33.4, 72.9)
Routing:
- net +3.3V: track 36.0 -> 38.6 mm
- net VCC: track 306.6 -> 307.5 mm
- net GND: vias 172 -> 173
