File: 3-phase/mainboard/3phaseDiverter - Copy.kicad_pcb (KiCad board)
At the start: 2 copper layers, 136.8 x 139.3 mm, 127 parts, among them CN9 SMA, IC1 ATmega328-P, IC2 LM358, J0 FTDI, J1 RESET, J10 D10, J11 D11, J12 D12, J13 D13, J16 D2, J17 D3, J18 D4, J19 D5, J2 D2, J21 D6, J22 D7, J23 D8, J24 D9, J25 D10, J26 D11, J27 D12, J28 D13, J3 D3, J30 OLED, J4 D4, J5 D5, J6 D6, J7 D7, J8 D8, J9 D9, U3 AP2112R5-3.3TRG1, X1 16MHz

Commit message: Some fixes
Parts:
- U3: footprint PCM_Package_TO_SOT_SMD_AKL:SOT-89-5_Handsoldering -> UserDef:AP2112R5-3.3TRG1_DIO
- moved C41 0.95 mm to (36.5, 47.2)
- moved C42 0.90 mm to (33.1, 42.2)
- moved C4 0.45 mm to (83.0, 40.2)
- moved U3 0.30 mm to (42.1, 44.8), turned to 0 degrees
- moved C40 0.19 mm to (47.1, 47.0)
- moved R5 0.12 mm to (50.0, 40.6)
- moved PS1 0.11 mm to (34.8, 91.2)
- turned REF4 to 0 degrees
Connections:
- C5 pad 1: GND -> AGND
- C6 pad 2: GND -> AGND
- D11 pad 2: GND -> AGND
- D12 pad 2: GND -> AGND
- D21 pad 2: GND -> AGND
- D22 pad 2: GND -> AGND
- D31 pad 2: GND -> AGND
- D32 pad 2: GND -> AGND
- IC1 pad 22: GND -> AGND
- PS1 pad 6: GND -> AGND
- REF1 pad 1: GND -> AGND
- REF3 pad 1: GND -> AGND
- REF4 pad 1: GND -> (no net)
Routing:
- net GND: track 246.9 -> 164.4 mm, vias 68 -> 16
- net AGND: track 0.00 -> 37.2 mm, vias 0 -> 48
- net Net-(IC2A-+): track 15.1 -> 13.5 mm
- net Net-(R41-Pad2): track 23.4 -> 22.0 mm
- net /D3: track 37.3 -> 36.1 mm
- net AREF: track 28.3 -> 27.1 mm
- net +5V: track 376.0 -> 375.0 mm
- net /D4: track 34.6 -> 34.0 mm
- added copper zone on B.Cu, net AGND
- added copper zone on F.Cu, net AGND
- removed copper zone on F.Cu, net GND
Other:
- board size 136.8 x 139.3 mm -> 136.8 x 140.8 mm
- board text added: "5V"
