File: 1-phase/Monophasé V4.4/untitled.kicad_sch (KiCad schematic)
At the start: 22 parts, among them CN1 Conn_02x07_Odd_Even, IC3 CD4543BE, IC4 74HC138N,652

Commit message: correction borne IC3 10
Connections:
- net at IC3.9 (7_SEGMENT_OUTPUTS_A), JP1.1 (A), R22.1: no longer IC3.10 (7_SEGMENT_OUTPUTS_B), JP1.2 (B), R16.1
- new net: IC3.10 (7_SEGMENT_OUTPUTS_B), JP1.2 (B), R16.1
Changed lines of the file:
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@@
   (junction (at 59.69 105.41) (diameter 0) (color 0 0 0 0)
   )
-  (junction (at 124.46 115.57) (diameter 0) (color 0 0 0 0)
-  )
   (junction (at 57.15 113.03) (diameter 0) (color 0 0 0 0)
   )
   (junction (at 77.47 68.58) (diameter 0) (color 0 0 0 0)
   )
+  (junction (at 133.35 113.03) (diameter 0) (color 0 0 0 0)
+  )
   (junction (at 125.73 107.95) (diameter 0) (color 0 0 0 0)
   )
@@
   (junction (at 147.32 97.79) (diameter 0) (color 0 0 0 0)
   )
-  (junction (at 124.46 113.03) (diameter 0) (color 0 0 0 0)
-  )
   (junction (at 127 105.41) (diameter 0) (color 0 0 0 0)
   )
@@
     (stroke (width 0) (type default))
   )
+  (wire (pts (xy 97.79 133.35) (xy 133.35 133.35))
+    (stroke (width 0) (type default))
+  )
   (wire (pts (xy 55.88 115.57) (xy 55.88 110.49))
     (stroke (width 0) (type default))
@@
     (stroke (width 0) (type default))
   )
-  (wire (pts (xy 124.46 113.03) (xy 146.05 113.03))
+  (wire (pts (xy 124.46 113.03) (xy 133.35 113.03))
     (stroke (width 0) (type default))
   )
@@
     (stroke (width 0) (type default))
   )
+  (wire (pts (xy 133.35 113.03) (xy 146.05 113.03))
+    (stroke (width 0) (type default))
+  )
   (wire (pts (xy 97.79 128.27) (xy 127 128.27))
     (stroke (width 0) (type default))
@@
     (stroke (width 0) (type default))
   )
+  (wire (pts (xy 133.35 133.35) (xy 133.35 113.03))
+    (stroke (width 0) (type default))
+  )
   (wire (pts (xy 134.62 81.28) (xy 134.62 110.49))
     (stroke (width 0) (type default))
@@
     (stroke (width 0) (type default))
   )
-  (wire (pts (xy 124.46 133.35) (xy 124.46 115.57))
-    (stroke (width 0) (type default))
-  )
   (wire (pts (xy 59.69 105.41) (xy 63.5 105.41))
     (stroke (width 0) (type default))
@@
     (stroke (width 0) (type default))
   )
-  (wire (pts (xy 97.79 133.35) (xy 124.46 133.35))
-    (stroke (width 0) (type default))
-  )
-  (wire (pts (xy 124.46 115.57) (xy 124.46 113.03))
-    (stroke (width 0) (type default))
-  )
