File: expansion_boards/ESP32/ESP32.kicad_sch (KiCad schematic)
At the start: 15 parts, among them J4 OLED, SW1 GPIO0, SW2 RESET, U1 ESP32-WROOM-32E

Commit message: Add AP2112R5A-3.3TRG1 3D model and update KiCad files
Added the AP2112R5A-3.3TRG1 STEP 3D model. Updated ESP32 and 3phaseDiverter KiCad project, schematic, PCB, and design rule files, including the addition of a new design rules file for the ESP32 board.
Parts:
- added C2, C3: 4u7, PCM_Capacitor_SMD_Handsoldering_AKL:C_1206_3216Metric_Pad1.42x1.75mm, symbol Device:C
- added JP2: SolderJumper_3_Open, Jumper:SolderJumper-3_P1.3mm_Open_Pad1.0x1.5mm_NumberLabels, symbol Jumper:SolderJumper_3_Open
- added U2: AP2112R5-3.3TRG1, PCM_Package_TO_SOT_SMD_AKL:Diodes_SOT-89-5, symbol UserDef:AP2112R5-3.3TRG1
- C1: value 10uF -> 100nF; footprint PCM_Capacitor_THT_AKL:C_Disc_D4.7mm_W2.5mm_P5.00mm -> PCM_Capacitor_SMD_Handsoldering_AKL:C_1206_3216Metric_Pad1.42x1.75mm
- LED1: value LED_3mm -> LED; footprint PCM_LED_THT_AKL:LED_D3.0mm -> PCM_LED_SMD_Handsoldering_AKL:LED_1206_3216Metric_Pad1.42x1.75mm
Connections:
- net GND: now also C2.2, C3.2, U2.2 (GND)
- net +5V: now reaches JP3.4 (Pin_4)
- net +5V: now also C2.1, JP2.2 (C), U2.4 (VIN)
- net +3.3V renamed +3V3
- net +3V3: now also C3.1, U2.5 (VOUT); no longer JP3.5 (Pin_5)
- new net: JP2.3 (B), U2.1 (NC)
- new net: JP2.1 (A), U2.3 (EN)

Commit message: Update ESP32 board UART connector and net assignments
Replaced JP1 pin header with pin socket, changed its position and orientation, and updated net assignments for UART pins. Adjusted net indices throughout the PCB to match schematic changes, updated silkscreen and fab layer properties, and modified JP3 socket position and labeling for consistency.
Parts:
- JP1: footprint Connector_PinHeader_2.54mm:PinHeader_1x06_P2.54mm_Vertical -> Connector_PinSocket_2.54mm:PinSocket_1x06_P2.54mm_Vertical
Connections:
- net +3V3: now also JP1.2 (Pin_2); no longer JP1.5 (Pin_5)
- net +5V: now also JP3.3 (Pin_3); no longer JP3.4 (Pin_4)
- net AVR_RX: now also JP3.4 (Pin_4); no longer JP3.3 (Pin_3)
- net AVR_TX: now also JP3.5 (Pin_5); no longer JP3.2 (Pin_2)
- net ESP_RX: now also JP1.4 (Pin_4); no longer JP1.3 (Pin_3)
- net ESP_TX: now also JP1.5 (Pin_5); no longer JP1.2 (Pin_2)
- net GND: now also JP1.1 (Pin_1), JP3.1 (Pin_1); no longer JP1.6 (Pin_6), JP3.6 (Pin_6)
