File: expansion_boards/mk2Wifi/mk2Wifi.kicad_sch (KiCad schematic)
At the start: 28 parts, among them J0 TRIG_EXT, J2 USB_C_Receptacle_USB2.0_16P, J3 UART_EXT, J4 OLED, SW1 SW_Push, U1 ESP32-C3-MINI-1, U2 AP2112K-3.3

Commit message: Fix split 3.3V power net on mk2Wifi OLED connector
J4 (OLED) VCC pin was on +3.3V (net 13) while the rest of the board
uses +3V3 (net 6), creating two separate unconnected power nets.
Changed #PWR6 to +3V3 in schematic and reassigned J4 pad 2 in PCB.

Co-Authored-By: Claude Opus 4.6 <noreply@anthropic.com>
Connections:
- net +3.3V is gone; now on net +3V3: J4.2 (VCC)
Changed lines of the file:
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@@
 	)
 	(junction
-		(at 118.11 31.75)
-		(diameter 0)
-		(color 0 0 0 0)
-	)
-	(junction
 		(at 135.89 34.29)
 		(diameter 0)
@@
 	(wire
 		(pts
-			(xy 118.11 30.48) (xy 118.11 31.75)
-		)
-		(stroke
-			(width 0)
-			(type default)
-		)
-	)
-	(wire
-		(pts
 			(xy 53.34 38.1) (xy 67.31 38.1)
 		)
@@
 	(wire
 		(pts
-			(xy 109.22 31.75) (xy 118.11 31.75)
+			(xy 109.22 31.75) (xy 119.38 31.75)
 		)
 		(stroke
@@
 	(wire
 		(pts
-			(xy 118.11 31.75) (xy 119.38 31.75)
-		)
-		(stroke
-			(width 0)
-			(type default)
-		)
-	)
-	(wire
-		(pts
 			(xy 24.13 55.88) (xy 24.13 58.42)
 		)
@@
 	)
 	(symbol
-		(lib_id "power:+3.3V")
+		(lib_id "power:+3V3")
 		(at 119.38 31.75 270)
 		(unit 1)
@@
 			)
 		)
-		(property "Value" "+3.3V"
+		(property "Value" "+3V3"
 			(at 123.19 31.7499 90)
 			(effects
@@
 			)
 		)
-		(property "Description" "Power symbol creates a global label with name \"+3.3V\""
+		(property "Description" "Power symbol creates a global label with name \"+3V3\""
 			(at 119.38 31.75 0)
 			(effects
@@
 					(unit 1)
 				)
-			)
-		)
-	)
-	(symbol
-		(lib_id "power:PWR_FLAG")
-		(at 118.11 30.48 0)
-		(unit 1)
-		(exclude_from_sim no)
-		(in_bom yes)
-		(on_board yes)
-		(dnp no)
-		(fields_autoplaced yes)
-		(property "Reference" "#FLG02"
-			(at 118.11 28.575 0)
-			(effects
-				(font
-					(size 1.27 1.27)
-				)
-				(hide yes)
-			)
-		)
-		(property "Value" "PWR_FLAG"
-			(at 120.65 29.2099 0)
-			(effects
-				(font
-					(size 1.27 1.27)
-				)
-				(justify left)
-			)
-		)
-		(property "Footprint" ""
-			(at 118.11 30.48 0)
-			(effects
-				(font
-					(size 1.27 1.27)
-				)
-				(hide yes)
-			)
-		)
-		(property "Datasheet" "~"
-			(at 118.11 30.48 0)
-			(effects
-				(font
-					(size 1.27 1.27)
-				)
-				(hide yes)
-			)
-		)
-		(property "Description" "Special symbol for telling ERC where power comes from"
-			(at 118.11 30.48 0)
-			(effects
-				(font
-					(size 1.27 1.27)
-				)
-				(hide yes)
-			)
-		)
-		(pin "1"
-		)
-		(instances
-			(project "mk2Wifi"
-				(path "/8f85e568-8005-4933-a5bc-4fca9da3c7b3"
-					(reference "#FLG02")
-					(unit 1)
-				)
