File: output_stage/Output_stage.kicad_sch (KiCad schematic)
At the start: 8 parts, among them J1 Conn_01x03_Socket, J2 Control/LED, J3 Control/LED, Q1 BTA41, U1 MOC3041M

Commit message: Add output_stage schematic description, SVG/PDF exports, and READMEs
- Add title block comments to output_stage schematic
- Export schematic as SVG and PDF
- Write full bilingual READMEs (FR/EN) with BOM, design notes, and clickable schematic

Co-Authored-By: Claude Opus 4.6 <noreply@anthropic.com>
Other:
- company: (none) -> Mk2PVRouter.com
Changed lines of the file:
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@@
     (date "2023-09-16")
     (rev "2.0")
+    (company "Mk2PVRouter.com")
+    (comment 1 "Triac power output stage for Mk2 PV Router")
+    (comment 2 "MOC3041M opto-triac — BTA41-600B power triac (41A / 600V)")
+    (comment 3 "Zero-crossing switching — Mains-isolated control input")
+    (comment 4 "License: CERN-OHL-S v2")
   )
   (junction (at 135.89 82.55) (diameter 0) (color 0 0 0 0)

Commit message: Update output_stage to MOC3043M and re-export schematic
- Migrate opto-triac from MOC3041M to MOC3043M (lower trigger current, Ift=5mA)
- Update READMEs and title block comment
- Re-export SVG and PDF

Co-Authored-By: Claude Opus 4.6 <noreply@anthropic.com>
Parts:
- U1: value MOC3041M -> MOC3043M; symbol Relay_SolidState:MOC3041M -> Relay_SolidState:MOC3043M
Changed lines of the file:
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@@
     (company "Mk2PVRouter.com")
     (comment 1 "Triac power output stage for Mk2 PV Router")
-    (comment 2 "MOC3041M opto-triac — BTA41-600B power triac (41A / 600V)")
+    (comment 2 "MOC3043M opto-triac — BTA41-600B power triac (41A / 600V)")
     (comment 3 "Zero-crossing switching — Mains-isolated control input")
     (comment 4 "License: CERN-OHL-S v2")
@@
     )
   )
-  (symbol (lib_id "Relay_SolidState:MOC3041M") (at 105.41 73.66 0) (unit 1)
+  (symbol (lib_id "Relay_SolidState:MOC3043M") (at 105.41 73.66 0) (unit 1)
     (in_bom yes) (on_board yes) (dnp no) (fields_autoplaced)
     (property "Reference" "U1" (at 105.41 66.04 0)
       (effects (font (size 1.27 1.27)))
     )
-    (property "Value" "MOC3041M" (at 105.41 68.58 0)
-      (effects (font (size 1.27 1.27)))
-    )
+    (property "Value" "MOC3043M" (at 105.41 68.58 0)
+      (effects (font (size 1.27 1.27)))
+    )

Commit message: Update output_stage: R1=220, MOC3063M notes, board images
- Change R1 from 120 to 220 ohm (sized for MOC3043M IFT=5mA, IF~10mA at 3.3V)
- Update schematic notes: 390 ohm for 5V, MOC3063M as 600V alternative
- Add board images (front, back, bare) to READMEs
- Re-export schematic SVG/PDF

Co-Authored-By: Claude Opus 4.6 <noreply@anthropic.com>
Parts:
- R1: value 120 -> 220
Other:
- note added: "Notes: 1. R1 = 220 Ohms for 3.3V supply (IF ~ 10 mA). For 5V supply, use R1 = 390 Ohms. 2. The power terminals at connector J1 can be interchanged. 3. When using a MOC3063M (600V, VDRM = 600V), change R2 from 330 to 360 Ohms."
- note removed: "Notes: 1. If the control signal comes from a 5V supply, R1 should be increased to 180 Ohms. 2. The power terminals at connector J1 can be interchanged. 3. When using a MOC3061M (600V), R2 should be changed to 360 Ohms."
