File: expansion_boards/mk2Wifi-C6/mk2Wifi-C6.kicad_pcb (KiCad board)
At the start: 2 copper layers, 51 x 26.3 mm, 32 parts, among them J0 TRIG_EXT, J2 USB_C_Receptacle_USB2.0_16P, J3 UART_EXT, J4 OLED, SW1 SW_Push, U1 ESP32-C6-MINI-1/U, U2 AP2112K-3.3

Commit message: Add MISC GPIO connector and update mk2Wifi-C6 docs
Add 5-pin MISC header (GPIO19-22) for additional user I/O.
Update readmes with complete strapping pin documentation (all 5 pins),
corrected UART GPIO mapping (GPIO16/GPIO17), new connector pinouts,
and regenerated schematic PDF/SVG. Rename UART_EXT connector to J0.

Co-Authored-By: Claude Opus 4.6 <noreply@anthropic.com>
Parts:
- added J4: MISC, Connector_PinHeader_2.54mm:PinHeader_1x05_P2.54mm_Vertical, F.Cu at (84.5, 58.6)
- SW1: value SW_Push -> Boot
- moved G004 15.6 mm to (68.5, 58.5)
- moved G*** 11.4 mm to (80.9, 55.5)
- moved SW1 1.01 mm to (96.2, 64.0)
- moved D1 0.72 mm to (89.1, 64.0)
- moved R2 0.72 mm to (87.7, 64.3)
- renumbered J3 to J0, J0 to J1, J4 to J3
Connections:
- U1 pad 25: unconnected-(U1-GPIO19-Pad25) -> /GPIO19
- U1 pad 26: unconnected-(U1-GPIO20-Pad26) -> /GPIO20
- U1 pad 27: unconnected-(U1-GPIO21-Pad27) -> /GPIO21
- U1 pad 28: unconnected-(U1-GPIO22-Pad28) -> /GPIO22
Routing:
- net /GPIO22: track 0.00 -> 14.5 mm
- net /GPIO21: track 0.00 -> 11.7 mm
- net /GPIO20: track 0.00 -> 8.81 mm
- net /GPIO19: track 0.00 -> 5.94 mm
- net /GPIO9: track 14.8 -> 15.8 mm
- net GND: vias 57 -> 62
Other:
- board text added: "19"
- board text added: "20"
- board text added: "21"
- board text added: "22"
